Commit message: feat: Add URDF for a burger delivery scene with Kinova robot components and its display launch file.

File: burger_description/urdf/delivery_scene_fixed.urdf (robot description, URDF)
Before this commit: robot burger_delivery_with_cars, 49 links, 50 joints
Links:
- link burger_grip_frame: geometry visual mesh filename=package://burger_description/meshes/arrow_pyramid_1m.stl scale=0.06 0.06 0.08; visual mesh filename=package://burger_description/meshes/arrow_pyramid_1m.stl scale=0.06 0.06 0.08
- link car1_base_link: geometry collision mesh filename=package://burger_description/visual/Carro2/meshes/base_link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; visual mesh filename=package://burger_description/meshes/arrow_pyramid_1m.stl scale=0.06 0.06 0.08
- link car2_base_link: geometry collision mesh filename=package://burger_description/visual/Carro4/meshes/base_link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; visual mesh filename=package://burger_description/meshes/arrow_pyramid_1m.stl scale=0.06 0.06 0.08
- link delivery_slot_1: geometry visual mesh filename=package://burger_description/meshes/arrow_pyramid_1m.stl scale=0.06 0.06 0.08; visual mesh filename=package://burger_description/meshes/arrow_pyramid_1m.stl scale=0.06 0.06 0.08
- link gen3_base_link: geometry collision mesh filename=package://burger_description/vendor/kortex_description/arms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; visual mesh filename=package://burger_description/vendor/kortex_description/arms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
- link gen3_bracelet_link: geometry collision mesh filename=package://burger_description/vendor/kortex_description/arms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; visual mesh filename=package://burger_description/vendor/kortex_description/arms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
- link gen3_forearm_link: geometry collision mesh filename=package://burger_description/vendor/kortex_description/arms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; visual mesh filename=package://burger_description/vendor/kortex_description/arms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
- link gen3_half_arm_1_link: geometry collision mesh filename=package://burger_description/vendor/kortex_description/arms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; visual mesh filename=package://burger_description/vendor/kortex_description/arms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
- link gen3_half_arm_2_link: geometry collision mesh filename=package://burger_description/vendor/kortex_description/arms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; visual mesh filename=package://burger_description/vendor/kortex_description/arms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
- link gen3_robotiq_85_base_link: geometry collision mesh filename=package://burger_description/vendor/robotiq_description/mes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; visual mesh filename=package://burger_description/vendor/robotiq_description/mes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
- link gen3_robotiq_85_left_finger_link: geometry collision mesh filename=package://burger_description/vendor/robotiq_description/mes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; visual mesh filename=package://burger_description/vendor/robotiq_description/mes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
- link gen3_robotiq_85_left_finger_tip_link: geometry collision mesh filename=package://burger_description/vendor/robotiq_description/mes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; visual mesh filename=package://burger_description/vendor/robotiq_description/mes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
- link gen3_robotiq_85_left_inner_knuckle_link: geometry collision mesh filename=package://burger_description/vendor/robotiq_description/mes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; visual mesh filename=package://burger_description/vendor/robotiq_description/mes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
- link gen3_robotiq_85_left_knuckle_link: geometry collision mesh filename=package://burger_description/vendor/robotiq_description/mes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; visual mesh filename=package://burger_description/vendor/robotiq_description/mes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
- link gen3_robotiq_85_right_finger_link: geometry collision mesh filename=package://burger_description/vendor/robotiq_description/mes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; visual mesh filename=package://burger_description/vendor/robotiq_description/mes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
- link gen3_robotiq_85_right_finger_tip_link: geometry collision mesh filename=package://burger_description/vendor/robotiq_description/mes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; visual mesh filename=package://burger_description/vendor/robotiq_description/mes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
- link gen3_robotiq_85_right_inner_knuckle_link: geometry collision mesh filename=package://burger_description/vendor/robotiq_description/mes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; visual mesh filename=package://burger_description/vendor/robotiq_description/mes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
- link gen3_robotiq_85_right_knuckle_link: geometry collision mesh filename=package://burger_description/vendor/robotiq_description/mes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; visual mesh filename=package://burger_description/vendor/robotiq_description/mes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
- link gen3_shoulder_link: geometry collision mesh filename=package://burger_description/vendor/kortex_description/arms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; visual mesh filename=package://burger_description/vendor/kortex_description/arms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
- link gen3_spherical_wrist_1_link: geometry collision mesh filename=package://burger_description/vendor/kortex_description/arms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; visual mesh filename=package://burger_description/vendor/kortex_description/arms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
- link gen3_spherical_wrist_2_link: geometry collision mesh filename=package://burger_description/vendor/kortex_description/arms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; visual mesh filename=package://burger_description/vendor/kortex_description/arms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
- link kinova_base_link: geometry visual mesh filename=package://burger_description/meshes/arrow_pyramid_1m.stl scale=0.06 0.06 0.08; visual mesh filename=package://burger_description/meshes/arrow_pyramid_1m.stl scale=0.06 0.06 0.08
- link kinova_tool_frame: geometry visual mesh filename=package://burger_description/meshes/arrow_pyramid_1m.stl scale=0.06 0.06 0.08; visual mesh filename=package://burger_description/meshes/arrow_pyramid_1m.stl scale=0.06 0.06 0.08
- link map: geometry visual mesh filename=package://burger_description/meshes/arrow_pyramid_1m.stl scale=0.06 0.06 0.08; visual mesh filename=package://burger_description/meshes/arrow_pyramid_1m.stl scale=0.06 0.06 0.08
- link overhead_camera_link: geometry visual mesh filename=package://burger_description/meshes/arrow_pyramid_1m.stl scale=0.06 0.06 0.08; visual mesh filename=package://burger_description/meshes/arrow_pyramid_1m.stl scale=0.06 0.06 0.08
- link staging_area: geometry visual mesh filename=package://burger_description/meshes/arrow_pyramid_1m.stl scale=0.06 0.06 0.08; visual mesh filename=package://burger_description/meshes/arrow_pyramid_1m.stl scale=0.06 0.06 0.08
- link table_link: geometry visual mesh filename=package://burger_description/meshes/arrow_pyramid_1m.stl scale=0.06 0.06 0.08; visual mesh filename=package://burger_description/meshes/arrow_pyramid_1m.stl scale=0.06 0.06 0.08
- link wrist_camera_mount_link: geometry collision box size=0.04 0.08 0.06; visual box size=0.04 0.08 0.06
Joints:
- joint map_to_camera: origin xyz=0.50 0.00 2.00 rpy=-1.5708 0 1.5708 -> xyz=2.00 1.00 1.50 rpy=0 0.5 -1.5708
- joint map_to_robot_a_base: child robot_a_base_link -> car1_base_link
- joint map_to_robot_b_base: child robot_b_base_link -> car2_base_link

Commit message: feat: implement dynamic visual localization system with AprilTags and update URDF models for improved camera integration.

File: burger_description/urdf/delivery_scene_fixed.urdf (robot description, URDF)
Before this commit: robot burger_delivery_with_cars, 49 links, 50 joints
Links:
- added link tag_mesa; visual box size=0.1 0.1 0.001
Joints:
- removed joint map_to_robot_a_base
- removed joint map_to_robot_b_base
- removed joint table_to_car1_base
- removed joint table_to_car2_base
- added joint table_to_tag_mesa: type fixed, parent table_link, child tag_mesa, origin xyz=0.5 0.3 0.025 rpy=0 0 0
