Commit message: feat: Add ROS 2 Jazzy installation script and burger_delivery_gen3 robot description package.

File: burger_description/urdf/burger_delivery_gen3.urdf (robot description, URDF)
Before this commit: robot burger_delivery_gen3, 43 links, 42 joints
Links:
- link wrist_camera_mount_link: geometry collision box size=0.04 0.08 0.06; visual box size=0.04 0.08 0.06

Commit message: urdf updated

File: burger_description/urdf/burger_delivery_gen3.urdf (robot description, URDF)
Before this commit: robot burger_delivery_gen3, 43 links, 42 joints
Joints:
- removed joint map_to_kinova_base
- removed joint map_to_world
- added joint table_to_kinova_base: type fixed, parent table_link, child kinova_base_link, origin xyz=1.20 0.30 0.5 rpy=0 0 0
- added joint table_to_world: type fixed, parent table_link, child world, origin xyz=0.20 0.30 0.00 rpy=0 0 0

File: burger_description/urdf/delivery_scene_fixed.urdf (robot description, URDF)
Before this commit: robot burger_delivery_with_cars, 50 links, 47 joints
Links:
- removed link car1_Base_rueda_castor_Link
- removed link car1_Rueda_castor_Link
- removed link car1_Rueda_derecha_Link
- removed link car1_Rueda_izquierda_Link
- removed link car1_base_link
- removed link car2_base_link
- removed link car2_wheel1
- removed link car2_wheel2
- removed link car2_wheel3
- removed link car2_wheel4
- link burger_grip_frame: mass None -> 0.1; geometry collision box size=0.04 0.08 0.02; visual mesh filename=package://burger_description/meshes/arrow_pyramid_1m.stl scale=0.06 0.06 0.08
- link delivery_slot_1: mass None -> 0.5; geometry collision box size=0.2 0.2 0.1; visual mesh filename=package://burger_description/meshes/arrow_pyramid_1m.stl scale=0.06 0.06 0.08
- link kinova_base_link: mass None -> 2.0; geometry collision box size=0.2 0.2 0.1; visual mesh filename=package://burger_description/meshes/arrow_pyramid_1m.stl scale=0.06 0.06 0.08
- link kinova_tool_frame: mass None -> 0.2; geometry collision box size=0.06 0.06 0.06; visual mesh filename=package://burger_description/meshes/arrow_pyramid_1m.stl scale=0.06 0.06 0.08
- link overhead_camera_link: mass None -> 0.2; geometry collision box size=0.05 0.05 0.05; visual mesh filename=package://burger_description/meshes/arrow_pyramid_1m.stl scale=0.06 0.06 0.08
- link staging_area: mass None -> 1.0; geometry collision box size=0.5 0.5 0.02; visual mesh filename=package://burger_description/meshes/arrow_pyramid_1m.stl scale=0.06 0.06 0.08
- link table_link: mass None -> 15.0; geometry collision box size=1.2 0.8 0.05; visual mesh filename=package://burger_description/meshes/arrow_pyramid_1m.stl scale=0.06 0.06 0.08
- link tag_mesa: mass None -> 0.01; geometry collision box size=0.1 0.1 0.001; visual box size=0.1 0.1 0.001
Joints:
- removed joint car1_Base_rueda_castor_Joint
- removed joint car1_Rueda_castor_Joint
- removed joint car1_Rueda_derecha_Joint
- removed joint car1_Rueda_izquierda_Joint
- removed joint car2_wheel1
- removed joint car2_wheel2
- removed joint car2_wheel3
- removed joint car2_wheel4
- removed joint map_to_kinova_base
- removed joint map_to_world
- added joint table_to_kinova_base: type fixed, parent table_link, child kinova_base_link, origin xyz=1.20 0.30 0.5 rpy=0 0 0
- added joint table_to_world: type fixed, parent table_link, child world, origin xyz=0.20 0.30 0.00 rpy=0 0 0

File: visual/burger_delivery_gen3.urdf (robot description, URDF)
Before this commit: robot burger_delivery_gen3, 43 links, 42 joints
Joints:
- removed joint map_to_kinova_base
- removed joint map_to_world
- added joint table_to_kinova_base: type fixed, parent table_link, child kinova_base_link, origin xyz=1.20 0.30 0.5 rpy=0 0 0
- added joint table_to_world: type fixed, parent table_link, child world, origin xyz=0.20 0.30 0.00 rpy=0 0 0
